Commit message: updates abv_chassis joint limits

File: src/abv_description/urdf/abv_chassis.urdf.xacro (robot description, xacro)
@@ -12,13 +12,13 @@
             <child link="x_link" />
             <axis xyz="1 0 0" />
-            <limit lower="0.0" upper="0.0" effort="0" velocity="10.0" />
+            <limit lower="-1.0" upper="1.0" effort="0" velocity="0.1" />
         </joint>
         <link name="x_link" />
-        <!-- Y translation -->
+        <!-- Y translation -->s
         <joint name="y_joint" type="prismatic">
             <parent link="x_link" />
             <child link="y_link" />
             <axis xyz="0 1 0" />
-            <limit lower="0.0" upper="0.0" effort="0" velocity="10.0" />
+            <limit lower="-1.0" upper="1.0" effort="0" velocity="0.1" />
         </joint>
         <link name="y_link" />
@@ -28,6 +28,5 @@
             <child link="vehicle_link" />
             <axis xyz="0 0 1" />
-            <limit lower="0" upper="0" effort="0" velocity="10.0" />
-            <!--limit lower="-3.14" upper="3.14" effort="0" velocity="10.0" /-->
+            <limit lower="-3.14" upper="3.14" effort="0" velocity="0.01" />
         </joint>
         <!-- Actual vehicle link with mesh -->

Commit message: updates to support ptera integration

File: src/abv_description/urdf/abv_chassis.urdf.xacro (robot description, xacro)
@@ -6,5 +6,17 @@
             <xacro:insert_block name="origin" />
         </joint>
-        <link name="base_link" />
+        <link name="base_link">
+            <inertial>
+                <mass value="0.001" />
+                <inertia
+                    ixx="0.001"
+                    ixy="0"
+                    ixz="0"
+                    iyy="0.001"
+                    iyz="0"
+                    izz="0.001"
+                />
+            </inertial>
+        </link>
         <!-- X translation -->
         <joint name="x_joint" type="prismatic">
@@ -14,6 +26,18 @@
             <limit lower="-1.0" upper="1.0" effort="0" velocity="0.1" />
         </joint>
-        <link name="x_link" />
-        <!-- Y translation -->s
+        <link name="x_link">
+            <inertial>
+                <mass value="0.001" />
+                <inertia
+                    ixx="0.001"
+                    ixy="0"
+                    ixz="0"
+                    iyy="0.001"
+                    iyz="0"
+                    izz="0.001"
+                />
+            </inertial>
+        </link>
+        <!-- Y translation -->
         <joint name="y_joint" type="prismatic">
             <parent link="x_link" />
@@ -22,5 +46,17 @@
             <limit lower="-1.0" upper="1.0" effort="0" velocity="0.1" />
         </joint>
-        <link name="y_link" />
+        <link name="y_link">
+            <inertial>
+                <mass value="0.001" />
+                <inertia
+                    ixx="0.001"
+                    ixy="0"
+                    ixz="0"
+                    iyy="0.001"
+                    iyz="0"
+                    izz="0.001"
+                />
+            </inertial>
+        </link>
         <!-- Yaw rotation -->
         <joint name="yaw_joint" type="revolute">
@@ -32,6 +68,17 @@
         <!-- Actual vehicle link with mesh -->
         <link name="vehicle_link">
+            <inertial>
+                <mass value="10.0" />
+                <inertia
+                    ixx="0.1"
+                    ixy="0"
+                    ixz="0"
+                    iyy="0.1"
+                    iyz="0"
+                    izz="0.1"
+                />
+            </inertial>
             <visual>
-            <origin xyz="-0.0175 -0.065 0.03" rpy="0 0 0" />
+                <origin xyz="-0.0175 -0.065 0.03" rpy="0 0 0" />
                 <geometry>
                     <mesh

File: src/abv_description/urdf/manipulators/widow_xl.urdf.xacro (robot description, xacro)
@@ -8,11 +8,19 @@
         </joint>
         <link name="${prefix}shoulder_mount">
+            <inertial>
+                <mass value="0.2"/>
+                <inertia ixx="0.0001" ixy="0.0" ixz="0.0"
+                         iyy="0.0001" iyz="0.0" izz="0.0001"/>
+            </inertial>
             <visual>
                 <geometry>
-                    <mesh
-                        filename="package://abv_description/meshes/widow-xl/shoulder_mount.dae"
-                    />
+                    <mesh filename="package://abv_description/meshes/widow-xl/shoulder_mount.dae"/>
                 </geometry>
             </visual>
+            <collision>
+                <geometry>
+                    <box size="0.07 0.07 0.05"/>
+                </geometry>
+            </collision>
         </link>
         <joint name="${prefix}shoulder_joint" type="revolute">
@@ -21,14 +29,25 @@
             <origin xyz="0.0 0.0 0.0" rpy="0 0 0" />
             <axis xyz="1 0 0" />
-            <limit lower="-1.57" upper="1.57" effort="0" velocity="1.0" />
+            <limit lower="-1.57" upper="1.57" effort="10" velocity="1.0" />
+            <dynamics damping="5.0" friction="0.5"/>
         </joint>
         <link name="${prefix}shoulder_link">
+            <inertial>
+                <mass value="0.3"/>
+                <origin xyz="0.0 -0.025 0.07" rpy="0 0 0"/>
+                <inertia ixx="0.0005" ixy="0.0" ixz="0.0"
+                         iyy="0.0005" iyz="0.0" izz="0.0001"/>
+            </inertial>
             <visual>
                 <geometry>
-                    <mesh
-                        filename="package://abv_description/meshes/widow-xl/shoulder.dae"
-                    />
+                    <mesh filename="package://abv_description/meshes/widow-xl/shoulder.dae"/>
                 </geometry>
             </visual>
+            <collision>
+                <origin xyz="0.0 -0.025 0.07" rpy="0 0 0"/>
+                <geometry>
+                    <cylinder radius="0.03" length="0.145"/>
+                </geometry>
+            </collision>
         </link>
         <joint name="${prefix}forearm_joint" type="revolute">
@@ -37,14 +56,25 @@
             <origin xyz="0.0 -0.0525 0.145" rpy="0 0 0" />
             <axis xyz="1 0 0" />
-            <limit lower="-1.57" upper="1.57" effort="0" velocity="1.0" />
+            <limit lower="-1.57" upper="1.57" effort="10" velocity="1.0" />
+            <dynamics damping="5.0" friction="0.5"/>
         </joint>
         <link name="${prefix}forearm_link">
+            <inertial>
+                <mass value="0.25"/>
+                <origin xyz="0.0 -0.075 0.0" rpy="0 0 0"/>
+                <inertia ixx="0.0005" ixy="0.0" ixz="0.0"
+                         iyy="0.0001" iyz="0.0" izz="0.0005"/>
+            </inertial>
             <visual>
                 <geometry>
-                    <mesh
-                        filename="package://abv_description/meshes/widow-xl/forearm.dae"
-                    />
+                    <mesh filename="package://abv_description/meshes/widow-xl/forearm.dae"/>
                 </geometry>
             </visual>
+            <collision>
+                <origin xyz="0.0 -0.075 0.0" rpy="0 0 0"/>
+                <geometry>
+                    <cylinder radius="0.025" length="0.15"/>
+                </geometry>
+            </collision>
         </link>
         <joint name="${prefix}wrist_joint" type="revolute">
@@ -53,14 +83,25 @@
             <origin xyz="0 -0.15 0" rpy="0 0 0" />
             <axis xyz="1 0 0" />
-            <limit lower="-1.57" upper="1.57" effort="0" velocity="1.0" />
+            <limit lower="-1.57" upper="1.57" effort="10" velocity="1.0" />
+            <dynamics damping="5.0" friction="0.5"/>
         </joint>
         <link name="${prefix}wrist_link">
+            <inertial>
+                <mass value="0.15"/>
+                <origin xyz="0.0 -0.0375 0.0" rpy="0 0 0"/>
+                <inertia ixx="0.0001" ixy="0.0" ixz="0.0"
+                         iyy="0.00005" iyz="0.0" izz="0.0001"/>
+            </inertial>
             <visual>
                 <geometry>
-                    <mesh
-                        filename="package://abv_description/meshes/widow-xl/wrist.dae"
-                    />
+                    <mesh filename="package://abv_description/meshes/widow-xl/wrist.dae"/>
                 </geometry>
             </visual>
+            <collision>
+                <origin xyz="0.0 -0.0375 0.0" rpy="0 0 0"/>
+                <geometry>
+                    <cylinder radius="0.02" length="0.075"/>
+                </geometry>
+            </collision>
         </link>
         <joint name="${prefix}wrist_rotate_joint" type="revolute">
@@ -69,14 +110,25 @@
             <origin xyz="0 -0.075 0" rpy="0 0 -1.57" />
             <axis xyz="1 0 0" />
-            <limit lower="-1.57" upper="1.57" effort="0" velocity="1.0" />
+            <limit lower="-1.57" upper="1.57" effort="10" velocity="1.0" />
+            <dynamics damping="5.0" friction="0.5"/>
         </joint>
         <link name="${prefix}wrist_rotate_link">
+            <inertial>
+                <mass value="0.1"/>
+                <origin xyz="0.02 0.0 0.0" rpy="0 0 0"/>
+                <inertia ixx="0.00005" ixy="0.0" ixz="0.0"
+                         iyy="0.00005" iyz="0.0" izz="0.00005"/>
+            </inertial>
             <visual>
                 <geometry>
-                    <mesh
-                        filename="package://abv_description/meshes/widow-xl/wrist_rotate.dae"
-                    />
+                    <mesh filename="package://abv_description/meshes/widow-xl/wrist_rotate.dae"/>
                 </geometry>
             </visual>
+            <collision>
+                <origin xyz="0.02 0.0 0.0" rpy="0 0 0"/>
+                <geometry>
+                    <cylinder radius="0.02" length="0.04"/>
+                </geometry>
+            </collision>
         </link>
         <joint name="${prefix}gripper_joint" type="fixed">
@@ -85,5 +137,6 @@
             <origin xyz="0.0575 0 0" rpy="0 0 0" />
         </joint>
-        <link name="${prefix}gripper_link" />
+        <!-- gripper_link is massless — mass accounted for in fingers -->
+        <link name="${prefix}gripper_link"/>
         <joint name="${prefix}left_finger_joint" type="prismatic">
             <parent link="${prefix}gripper_link" />
@@ -92,14 +145,23 @@
             <axis xyz="0 -1 0" />
             <limit lower="0.0" upper="0.0325" effort="10" velocity="1.0" />
+            <dynamics damping="5.0" friction="0.5"/>
         </joint>
         <link name="${prefix}left_finger_link">
+            <inertial>
+                <mass value="0.05"/>
+                <inertia ixx="0.00001" ixy="0.0" ixz="0.0"
+                         iyy="0.00001" iyz="0.0" izz="0.00001"/>
+            </inertial>
             <visual>
                 <origin xyz="0 0 0" rpy="0 0 1.57" />
                 <geometry>
-                    <mesh
-                        filename="package://abv_description/meshes/widow-xl/finger.dae"
-                    />
+                    <mesh filename="package://abv_description/meshes/widow-xl/finger.dae"/>
                 </geometry>
             </visual>
+            <collision>
+                <geometry>
+                    <box size="0.015 0.03 0.04"/>
+                </geometry>
+            </collision>
         </link>
         <joint name="${prefix}right_finger_joint" type="prismatic">
@@ -109,14 +171,23 @@
             <axis xyz="0 1 0" />
             <limit lower="0.0" upper="0.0325" effort="10" velocity="1.0" />
+            <dynamics damping="5.0" friction="0.5"/>
         </joint>
         <link name="${prefix}right_finger_link">
+            <inertial>
+                <mass value="0.05"/>
+                <inertia ixx="0.00001" ixy="0.0" ixz="0.0"
+                         iyy="0.00001" iyz="0.0" izz="0.00001"/>
+            </inertial>
             <visual>
                 <origin xyz="0 0 0" rpy="3.14159 0 -1.57" />
                 <geometry>
-                    <mesh
-                        filename="package://abv_description/meshes/widow-xl/finger.dae"
-                    />
+                    <mesh filename="package://abv_description/meshes/widow-xl/finger.dae"/>
                 </geometry>
             </visual>
+            <collision>
+                <geometry>
+                    <box size="0.015 0.03 0.04"/>
+                </geometry>
+            </collision>
         </link>
     </xacro:macro>
